File: ECE_196_proj_shem/ECE_196_proj_shem-backups/ECE_196_proj_shem-2024-04-28_200304/ECE_196_proj_shem.kicad_sch (KiCad schematic)
At the start: 12 parts, among them J1 Screw_Terminal_01x05, U1 MAX9814

Commit message: Updating images.
Parts:
- removed FB1, FB2: FerriteBead_Small, symbol Device:FerriteBead_Small
- removed J1: Screw_Terminal_01x05, symbol Connector:Screw_Terminal_01x05
- added FB1, FB3: FerriteBead, Ferrite_THT:LairdTech_28C0236-0JW-10, symbol Device:FerriteBead
- added J2: Screw_Terminal_01x06, Connector_PinHeader_1.27mm:PinHeader_1x06_P1.27mm_Vertical, symbol Connector:Screw_Terminal_01x06
- added MK1: CMA-4544PF-W, CMA-4544PF-W:MIC_CMA-4544PF-W, symbol CMA-4544PF-W:CMA-4544PF-W
- C1, C2, C3, C4, C5: footprint (none) -> Capacitor_SMD:C_1825_4564Metric
- R1, R2, R4: footprint (none) -> Resistor_SMD:R_2512_6332Metric
Connections:
- net A/R: now also J2.5 (Pin_5)
- net GAIN: now also J2.3 (Pin_3)
- net GND: now also FB1.2, MK1.1
- net OUTPUT: now also J2.4 (Pin_4)
- net VDD: now also FB3.2, J2.6 (Pin_6)
- net CMA-4544PF_W: no longer names the net of C5.2, R1.2
- net CMA-4544PF_W: now also MK1.2
- new net: FB1.1, J2.1 (Pin_1)
- new net: FB3.1, J2.2 (Pin_2)
- no-connect marks 0 -> 1
Other:
- moved on the sheet: C4

Commit message: Adding these files for backup.
Parts:
- removed FB1, FB3: FerriteBead, Ferrite_THT:LairdTech_28C0236-0JW-10, symbol Device:FerriteBead
- removed J2: Screw_Terminal_01x06, Connector_PinHeader_1.27mm:PinHeader_1x06_P1.27mm_Vertical, symbol Connector:Screw_Terminal_01x06
- added J1: Screw_Terminal_01x05, Connector_PinHeader_1.27mm:PinHeader_1x05_P1.27mm_Vertical, symbol Connector:Screw_Terminal_01x05
- C1: value 0.1uF -> 470nF; footprint Capacitor_SMD:C_1825_4564Metric -> Capacitor_SMD:C_0504_1310Metric
- C2: value 22uF -> 2.2uF; footprint Capacitor_SMD:C_1825_4564Metric -> Capacitor_SMD:C_0504_1310Metric
- C3, C5: footprint Capacitor_SMD:C_1825_4564Metric -> Capacitor_SMD:C_0504_1310Metric
- C4: value 2.2uF -> 1uF; footprint Capacitor_SMD:C_1825_4564Metric -> Capacitor_SMD:C_0504_1310Metric
- R1: value 22k -> 2.2k; footprint Resistor_SMD:R_2512_6332Metric -> Resistor_SMD:R_0603_1608Metric
- R2, R4: footprint Resistor_SMD:R_2512_6332Metric -> Resistor_SMD:R_0603_1608Metric
Connections:
- net A/R is gone; now on net GND: U1.9 (A/R)
- net VDD is gone; now on net GAIN: C4.1, U1.2 (~{SHDN}), U1.5 (VDD)
- net GAIN: now also J1.2 (Pin_2), J1.3 (Pin_3)
- net GND: now also J1.1 (Pin_1), J1.5 (Pin_5)
- net OUTPUT: now also J1.4 (Pin_4)
